File: handheld-sstc.kicad_sch (KiCad schematic)
At the start: 67 parts, among them J1 Ext 15V in, J2 Ext 15V out, J3 Secondary Bottom, J4 Pri-, J5 Pri+, J6 Main power (20A max), J7 CT input, Q1 IPP320N20N3, Q2 IPP320N20N3, Q3 IPP320N20N3, SW1 SW_SPDT, SW2 SW_SPDT, U1 UCC27624V, U2 TLC555xP, U3 LM2596T-ADJ, U4 LM7815_TO220

Commit message: Fix some small problems on PCB, add screenshots and some text
Connections:
- net Drain: now also D4.1 (K); no longer D4.2 (A)
- net GND: now also D4.2 (A); no longer D4.1 (K)
Other:
- moved on the sheet: D4
Changed lines of the file:
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@@
 	(symbol
 		(lib_id "Device:D_Zener")
-		(at 250.19 106.68 90)
+		(at 250.19 106.68 270)
 		(unit 1)
 		(exclude_from_sim no)
@@
 					(size 1.27 1.27)
 				)
-				(justify right)
+				(justify left)
 			)
 		)
@@
 					(size 1.27 1.27)
 				)
-				(justify right)
+				(justify left)
 			)
 		)
