File: handheld-sstc.kicad_pcb (KiCad board)
At the start: 2 copper layers, 180 x 58 mm, 64 parts, among them J1 Ext 15V in, J2 Ext 15V out, J3 Secondary Bottom, J4 Pri-, J5 Pri+, J6 Main power, J7 CT input, Q1 IPP320N20N3, Q2 IPP320N20N3, Q3 IPP320N20N3, SW1 SW_SPDT, SW2 Trigger, U1 UCC27624V, U2 TLC555CP, U3 LM2596T-ADJ, U4 LM7815_TO220

Commit message: Fix clearances and add some text
Parts:
- added G***: LOGO, LOGO, B.Cu at (201.5, 120.7)
Routing:
- net GND: vias 157 -> 163
Other:
- board text added: "Don't touch energized or grounded metal when using handheld"
- board text added: "Project files and BOM on GitHub: https://github.com/penguinmoose/handheld-sstc"
- board text added: "RF burn hazard!"

Commit message: Fix some small problems on PCB, add screenshots and some text
Parts:
- added G***: LOGO, LOGO, B.Cu at (77.5, 83.0)
- C12: value .33u -> 0.33u
- C3: value 2.2u PP Film 630VDC -> 2.2u
- C4: value 47n film 1kVdc -> 47n
- J6: value Main power -> Main power (20A max)
- JP1: value 15V enable> -> 15V enable
- R1: value 331 -> 330Ω
- R9: footprint Resistor_THT:R_Axial_DIN0207_L6.3mm_D2.5mm_P7.62mm_Horizontal -> Resistor_THT:R_Axial_DIN0207_L6.3mm_D2.5mm_P10.16mm_Horizontal
- RV1: value off-time -> 50k
- RV2: value on-time -> 5k
- SW2: value Trigger -> SW_SPDT
- TP1: value Interruption sig -> Interruption signal
- U2: value TLC555CP -> TLC555xP
- turned D4 to -90 degrees
Connections:
- D4 pad 1: GND -> Drain
- D4 pad 2: Drain -> GND
Routing:
- net 555_thr: track 26.3 -> 50.5 mm
- net Net-(D10-K): track 9.62 -> 21.2 mm
- net gd_ena: track 12.7 -> 23.3 mm, vias 2 -> 4
- net R9-RV1: track 7.53 -> 8.63 mm
Other:
- board text added: "Handheld SSTC v1.7 created and designed by Johannes ©2026 7/9/2026"
- board text added: "Project files and BOM on GitHub (CC BY-NC-SA): https://github.com/penguinmoose/handheld-sstc"
- board text added: "← Signal and gate-drive section"
- board text removed: "Project files and BOM on GitHub: https://github.com/penguinmoose/handheld-sstc"

Commit message: Add gerber files and minor edits
Parts:
- TP1: value Interruption signal -> Interruption sig.
Routing:
- net Drain: track 88.8 -> 122.8 mm
- net VBUS: track 151.3 -> 183.9 mm
- net GND: track 2.65 -> 5.35 mm, vias 163 -> 165
- net +15V: track 167.7 -> 169.3 mm, vias 4 -> 3
- net VCC: track 16.0 -> 15.1 mm
- net gd_ena: track 23.3 -> 24.1 mm
